File: mcu.kicad_sch (KiCad schematic)
At the start: 33 parts, among them U1 STM32H723VGTx, U13 BMI323, U14 AS5047P-ATST, U15 TCAN1044VDRQ1, X1 8MHz

Commit message: WiP layout
Connections:
- net +3V3: now also R7.2
- net GND: no longer R7.2
- net VBUS: no longer names the net of U1.68 (PA9)
Changed lines of the file:
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@@
 	(text "Basic I/O, place it last"
 		(exclude_from_sim no)
-		(at 27.686 84.582 0)
+		(at 27.686 93.218 0)
 		(effects
 			(font
@@
 	)
 	(junction
-		(at 199.39 116.84)
-		(diameter 0)
-		(color 0 0 0 0)
-	)
-	(junction
 		(at 25.4 63.5)
 		(diameter 0)
@@
 	)
 	(junction
+		(at 199.39 116.84)
+		(diameter 0)
+		(color 0 0 0 0)
+	)
+	(junction
 		(at 160.02 80.01)
 		(diameter 0)
@@
 	)
 	(no_connect
-		(at 27.94 93.98)
+		(at 29.21 100.33)
 	)
 	(no_connect
@@
 	)
 	(no_connect
-		(at 29.21 88.9)
+		(at 29.21 95.25)
 	)
 	(no_connect
@@
 	)
 	(no_connect
-		(at 27.94 96.52)
+		(at 29.21 102.87)
 	)
 	(no_connect
@@
 	)
 	(no_connect
-		(at 29.21 91.44)
+		(at 29.21 97.79)
 	)
 	(no_connect
@@
 	)
 	(no_connect
-		(at 33.02 77.47)
+		(at 30.48 86.36)
 	)
 	(no_connect
@@
 	(wire
 		(pts
-			(xy 199.39 118.11) (xy 199.39 116.84)
-		)
-		(stroke
-			(width 0)
-			(type default)
-		)
-	)
-	(wire
-		(pts
 			(xy 255.27 101.6) (xy 255.27 106.68)
 		)
@@
 	(wire
 		(pts
-			(xy 199.39 116.84) (xy 217.17 116.84)
-		)
-		(stroke
-			(width 0)
-			(type default)
-		)
-	)
-	(wire
-		(pts
 			(xy 116.84 69.85) (xy 121.92 69.85)
 		)
@@
 	(wire
 		(pts
+			(xy 199.39 116.84) (xy 217.17 116.84)
+		)
+		(stroke
+			(width 0)
+			(type default)
+		)
+	)
+	(wire
+		(pts
 			(xy 52.07 74.93) (xy 55.88 74.93)
 		)
@@
 	(wire
 		(pts
+			(xy 199.39 115.57) (xy 199.39 116.84)
+		)
+		(stroke
+			(width 0)
+			(type default)
+		)
+	)
+	(wire
+		(pts
 			(xy 46.99 146.05) (xy 46.99 143.51)
 		)
@@
 	(wire
 		(pts
-			(xy 116.84 54.61) (xy 121.92 54.61)
-		)
-		(stroke
-			(width 0)
-			(type default)
-		)
-	)
-	(wire
-		(pts
 			(xy 26.67 173.99) (xy 34.29 173.99)
 		)
@@
 	(wire
 		(pts
+			(xy 199.39 101.6) (xy 199.39 107.95)
+		)
+		(stroke
+			(width 0)
+			(type default)
+		)
+	)
+	(wire
+		(pts
 			(xy 104.14 173.99) (xy 111.76 173.99)
 		)
@@
 	(global_label "USR_BTN2"
 		(shape input)
-		(at 29.21 91.44 180)
+		(at 29.21 97.79 180)
 		(fields_autoplaced yes)
 		(effects
@@
 		)
 		(property "Intersheetrefs" "${INTERSHEET_REFS}"
-			(at 16.6696 91.44 0)
+			(at 16.6696 97.79 0)
 			(effects
 				(font
@@
 	(global_label "IMU_INT1"
 		(shape input)
-		(at 27.94 93.98 180)
+		(at 29.21 100.33 180)
 		(fields_autoplaced yes)
 		(effects
@@
 		)
 		(property "Intersheetrefs" "${INTERSHEET_REFS}"
-			(at 16.4881 93.98 0)
+			(at 17.7581 100.33 0)
 			(effects
 				(font
@@
 	(global_label "USR_BTN1"
 		(shape input)
-		(at 29.21 88.9 180)
+		(at 29.21 95.25 180)
 		(fields_autoplaced yes)
 		(effects
@@
 		)
 		(property "Intersheetrefs" "${INTERSHEET_REFS}"
-			(at 16.6696 88.9 0)
+			(at 16.6696 95.25 0)
 			(effects
 				(font
@@
 	(global_label "IMU_INT2"
 		(shape input)
-		(at 27.94 96.52 180)
+		(at 29.21 102.87 180)
 		(fields_autoplaced yes)
 		(effects
@@
 		)
 		(property "Intersheetrefs" "${INTERSHEET_REFS}"
-			(at 16.4881 96.52 0)
+			(at 17.7581 102.87 0)
 			(effects
 				(font
@@
 	(hierarchical_label "EN_FILTER_U"
 		(shape output)
-		(at 33.02 77.47 180)
+		(at 30.48 86.36 180)
 		(effects
 			(font
@@
 	(hierarchical_label "OCP_V_N"
 		(shape input)
-		(at 29.21 118.11 180)
+		(at 26.67 124.46 180)
 		(effects
 			(font
@@
 	(hierarchical_label "OCP_V_P"
 		(shape input)
-		(at 29.21 115.57 180)
+		(at 26.67 121.92 180)
 		(effects
 			(font
@@
 	(hierarchical_label "HALL1"
 		(shape input)
-		(at 20.32 100.33 180)
+		(at 24.13 109.22 180)
 		(effects
 			(font
@@
 	(hierarchical_label "OCP_U_N"
 		(shape input)
-		(at 29.21 113.03 180)
+		(at 26.67 119.38 180)
 		(effects
 			(font
@@
 	(hierarchical_label "OCP_U_P"
 		(shape input)
-		(at 29.21 110.49 180)
+		(at 26.67 116.84 180)
 		(effects
 			(font
@@
 	(hierarchical_label "OCP_W_P"
 		(shape input)
-		(at 29.21 120.65 180)
+		(at 26.67 127 180)
 		(effects
 			(font
@@
 	(hierarchical_label "HALL3"
 		(shape input)
-		(at 20.32 105.41 180)
+		(at 24.13 114.3 180)
 		(effects
 			(font
@@
 		)
 	)
-	(hierarchical_label "VBUS"
-		(shape input)
-		(at 121.92 54.61 0)
-		(effects
-			(font
-				(size 1.27 1.27)
-			)
-			(justify left)
-		)
-	)
 	(hierarchical_label "HALL2"
 		(shape input)
-		(at 20.32 102.87 180)
+		(at 24.13 111.76 180)
 		(effects
 			(font
@@
 	(hierarchical_label "OCP_W_N"
 		(shape input)
-		(at 29.21 123.19 180)
+		(at 26.67 129.54 180)
 		(effects
 			(font
@@
 	)
 	(symbol
-		(lib_id "power:GND")
-		(at 199.39 125.73 0)
-		(unit 1)
-		(exclude_from_sim no)
-		(in_bom yes)
-		(on_board yes)
-		(dnp no)
-		(property "Reference" "#PWR0106"
-			(at 199.39 132.08 0)
-			(effects
-				(font
-					(size 1.27 1.27)
-				)
-				(hide yes)
-			)
-		)
-		(property "Value" "GND"
-			(at 199.39 129.794 0)
-			(effects
-				(font
-					(size 1.27 1.27)
-				)
-			)
-		)
-		(property "Footprint" ""
-			(at 199.39 125.73 0)
-			(effects
-				(font
-					(size 1.27 1.27)
-				)
-				(hide yes)
-			)
-		)
-		(property "Datasheet" ""
-			(at 199.39 125.73 0)
-			(effects
-				(font
-					(size 1.27 1.27)
-				)
-				(hide yes)
-			)
-		)
-		(property "Description" "Power symbol creates a global label with name \"GND\" , ground"
-			(at 199.39 125.73 0)
-			(effects
-				(font
-					(size 1.27 1.27)
-				)
-				(hide yes)
-			)
-		)
-		(pin "1"
-		)
-		(instances
-			(project "NanoGaN"
-				(path "/aa8a494f-605e-4a00-9d3c-daec94709fcb/ac0a01b7-48dd-40d5-85d0-d2ed24ad85a4"
-					(reference "#PWR0106")
-					(unit 1)
-				)
-			)
-		)
-	)
-	(symbol
 		(lib_id "Device:C")
 		(at 41.91 179.07 0)
@@
 		(on_board yes)
 		(dnp no)
-		(fields_autoplaced yes)
 		(property "Reference" "#PWR0101"
 			(at 214.63 105.41 0)
@@
 	)
 	(symbol
+		(lib_id "power:+3V3")
+		(at 199.39 101.6 0)
+		(unit 1)
+		(exclude_from_sim no)
+		(in_bom yes)
+		(on_board yes)
+		(dnp no)
+		(property "Reference" "#PWR0106"
+			(at 199.39 105.41 0)
+			(effects
+				(font
+					(size 1.27 1.27)
+				)
+				(hide yes)
+			)
+		)
+		(property "Value" "+3V3"
+			(at 199.39 96.52 0)
+			(effects
+				(font
+					(size 1.27 1.27)
+				)
+			)
+		)
+		(property "Footprint" ""
+			(at 199.39 101.6 0)
+			(effects
+				(font
+					(size 1.27 1.27)
+				)
+				(hide yes)
+			)
+		)
+		(property "Datasheet" ""
+			(at 199.39 101.6 0)
+			(effects
+				(font
+					(size 1.27 1.27)
+				)
+				(hide yes)
+			)
+		)
+		(property "Description" "Power symbol creates a global label with name \"+3V3\""
+			(at 199.39 101.6 0)
+			(effects
+				(font
+					(size 1.27 1.27)
+				)
+				(hide yes)
+			)
+		)
+		(pin "1"
+		)
+		(instances
+			(project "NanoGaN"
+				(path "/aa8a494f-605e-4a00-9d3c-daec94709fcb/ac0a01b7-48dd-40d5-85d0-d2ed24ad85a4"
+					(reference "#PWR0106")
+					(unit 1)
+				)
+			)
+		)
+	)
+	(symbol
 		(lib_id "Device:C")
 		(at 172.72 144.78 0)
@@
 	(symbol
 		(lib_id "Device:R")
-		(at 199.39 121.92 0)
+		(at 199.39 111.76 180)
 		(unit 1)
 		(exclude_from_sim no)
@@
 		(dnp no)
 		(property "Reference" "R7"
-			(at 201.422 121.92 90)
+			(at 197.358 111.76 90)
 			(effects
 				(font
@@
 		)
 		(property "Value" "10k"
-			(at 199.39 121.92 90)
+			(at 199.39 111.76 90)
 			(effects
 				(font
@@
 		)
 		(property "Footprint" "Resistor_SMD:R_0402_1005Metric"
-			(at 197.612 121.92 90)
+			(at 201.168 111.76 90)
 			(effects
 				(font
@@
 		)
 		(property "Datasheet" "~"
-			(at 199.39 121.92 0)
+			(at 199.39 111.76 0)
 			(effects
 				(font
@@
 		)
 		(property "Description" "-55℃~+155℃ 10kΩ 50V 62.5mW Thick Film Resistor ±1% ±100ppm/℃ 0402 Chip Resistor - Surface Mount ROHS"
-			(at 199.39 121.92 0)
+			(at 199.39 111.76 0)
 			(effects
 				(font
@@
 		)
 		(property "LCSC" "C25744"
-			(at 199.39 121.92 0)
+			(at 199.39 111.76 0)
 			(effects
 				(font
