File: mcu.kicad_sch (KiCad schematic)
At the start: 33 parts, among them U1 STM32H723VGTx, U13 BMI323, U14 AS5047P-ATST, U15 TCAN1044VDRQ1, X1 8MHz

Commit message: added the first draft of the layout
Parts:
- removed R7: 10k, Resistor_SMD:R_0402_1005Metric, symbol Device:R
- added C94, C95: 1n, Capacitor_SMD:C_0201_0603Metric, symbol Device:C
Connections:
- net AGND: now also C94.2, C95.2
- net DAC_OCP_N: now also C95.1
- net DAC_OCP_P: now also C94.1
- net FAN_PWM: no longer U1.96 (PB9)
- net FDCAN1_RX: now also U1.95 (PB8); no longer U1.81 (PD0)
- net FDCAN1_STB: now also U1.85 (PD4); no longer U1.83 (PD2)
- net FDCAN1_TX: now also U1.96 (PB9); no longer U1.82 (PD1)
- net HALL1: now also U1.7 (PC13)
- net HALL2: now also U1.8 (PC14)
- net HALL3: now also U1.9 (PC15)
- net SERVO: no longer U1.90 (PB4(NJTRST)), U1.91 (PB5)
- net SPI2_MISO: now also U13.1 (SDO); no longer U14.3 (MISO)
- net SPI2_MOSI: now also U13.14 (SDX); no longer U14.4 (MOSI)
- net SPI2_NSS: now also U13.12 (CSB); no longer U14.1 (CSn)
- net SPI2_SCK: now also U13.13 (SCX); no longer U14.2 (CLK)
- net SPI4_MISO: now also U14.3 (MISO); no longer U13.1 (SDO)
- net SPI4_MOSI: now also U14.4 (MOSI); no longer U13.14 (SDX)
- net SPI4_NSS: now also U14.1 (CSn); no longer U13.12 (CSB)
- net SPI4_SCK: now also U14.2 (CLK); no longer U13.13 (SCX)
- net U_PHASE_SENS_U: now also U1.22 (PA0); no longer U1.35 (PB1)
- net U_PHASE_SENS_V: now also U1.23 (PA1); no longer U1.32 (PC4)
- net U_PHASE_SENS_W: now also U1.24 (PA2); no longer U1.31 (PA7)
- net EN_FILTER_I: no longer names the net of U1.37 (PE7)
- net I_CURR_SENS_U renamed I_CURR_SENS_W-
- net I_CURR_SENS_V renamed I_CURR_SENS_V-
- net I_CURR_SENS_W renamed I_CURR_SENS_U+
- net USART1_RX: no longer names the net of U1.93 (PB7)
- net USART1_TX: no longer names the net of U1.92 (PB6)
- new net I_CURR_SENS_U-: U1.31 (PA7)
- new net I_CURR_SENS_V+: U1.32 (PC4)
- new net I_CURR_SENS_W+: U1.35 (PB1)
- new net UART4_RX: U1.81 (PD0)
- new net UART4_TX: U1.82 (PD1)
- no-connect marks 46 -> 42

Commit message: wip layout
Parts:
- removed C79, C93: 1u, Capacitor_SMD:C_0402_1005Metric, symbol Device:C
- C58: footprint Capacitor_SMD:C_0402_1005Metric -> Capacitor_SMD:C_0603_1608Metric_Pad1.08x0.95mm_HandSolder; LCSC C307427 -> (none)
- C59: footprint Capacitor_SMD:C_0402_1005Metric -> Capacitor_SMD:C_0603_1608Metric_Pad1.08x0.95mm_HandSolder; LCSC C424821 -> (none)
- C94, C95: now not fitted; now left out of the parts list
Connections:
- net AGND: no longer C95.2
- net GATE_U_HI: now also U1.43 (PE13); no longer U1.39 (PE9)
- net GATE_U_LI: now also U1.42 (PE12); no longer U1.38 (PE8)
- net GATE_W_HI: now also U1.39 (PE9); no longer U1.43 (PE13)
- net GATE_W_LI: now also U1.38 (PE8); no longer U1.42 (PE12)
- net GND: now also C95.2

Commit message: wip layout
Connections:
- net GATE_U_HI renamed GATE_U+
- net GATE_U_LI renamed GATE_U-
- net GATE_V_HI renamed GATE_V+
- net GATE_V_LI renamed GATE_V-
- net GATE_W_HI renamed GATE_W+
- net GATE_W_LI renamed GATE_W-
Changed lines of the file:
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@@
 		)
 	)
-	(hierarchical_label "GATE_W_HI"
+	(hierarchical_label "GATE_W+"
 		(shape output)
 		(at 52.07 77.47 180)
@@
 		)
 	)
-	(hierarchical_label "GATE_V_LI"
+	(hierarchical_label "GATE_V-"
 		(shape output)
 		(at 52.07 80.01 180)
@@
 		)
 	)
-	(hierarchical_label "GATE_V_HI"
+	(hierarchical_label "GATE_V+"
 		(shape output)
 		(at 52.07 82.55 180)
@@
 		)
 	)
-	(hierarchical_label "GATE_U_LI"
+	(hierarchical_label "GATE_U-"
 		(shape output)
 		(at 52.07 85.09 180)
@@
 		)
 	)
-	(hierarchical_label "GATE_U_HI"
+	(hierarchical_label "GATE_U+"
 		(shape output)
 		(at 52.07 87.63 180)
@@
 		)
 	)
-	(hierarchical_label "GATE_W_LI"
+	(hierarchical_label "GATE_W-"
 		(shape output)
 		(at 52.07 74.93 180)

Commit message: wip layout
Connections:
- net I_CURR_SENS_U+: now also U1.34 (PB0); no longer U1.30 (PA6)
- net I_CURR_SENS_U-: now also U1.35 (PB1); no longer U1.31 (PA7)
- net I_CURR_SENS_W+: now also U1.30 (PA6); no longer U1.35 (PB1)
- net I_CURR_SENS_W-: now also U1.31 (PA7); no longer U1.34 (PB0)

Commit message: first draft of the PCB
Connections:
- net AGND: no longer C72.2, C80.2, U1.19 (VSSA)
- net FAN_PWM: now also U1.46 (PB10)
- net GND: now also C72.2, C80.2, U1.19 (VSSA)
- net IMU_INT1: now also U1.97 (PE0)
- net OCP_U_N: now also U1.87 (PD6)
- net OCP_U_P: now also U1.86 (PD5)
- net OCP_V_N: now also U1.55 (PD8)
- net OCP_V_P: now also U1.88 (PD7)
- net OCP_W_N: now also U1.57 (PD10)
- net OCP_W_P: now also U1.56 (PD9)
- net SERVO: now also U1.59 (PD12)
- net SPI2_MISO: now also U14.3 (MISO); no longer U13.1 (SDO)
- net SPI2_MOSI: now also U14.4 (MOSI); no longer U13.14 (SDX)
- net SPI2_NSS: now also U14.1 (CSn); no longer U13.12 (CSB)
- net SPI2_SCK: now also U14.2 (CLK); no longer U13.13 (SCX)
- net SPI4_MISO: now also U13.1 (SDO); no longer U14.3 (MISO)
- net SPI4_MOSI: now also U13.14 (SDX); no longer U14.4 (MOSI)
- net SPI4_NSS: now also U13.12 (CSB); no longer U14.1 (CSn)
- net SPI4_SCK: now also U13.13 (SCX); no longer U14.2 (CLK)
- net U_PHASE_SENS_U: now also U1.24 (PA2); no longer U1.22 (PA0)
- net U_PHASE_SENS_W: now also U1.22 (PA0); no longer U1.24 (PA2)
- net IMU_INT2: no longer names the net of U13.9 (INT2)
- no-connect marks 42 -> 32
Other:
- note removed: "Basic I/O, place it last"
- note removed: "is it okay X5R?"
- note removed: "maybe chose different xtal?"

Commit message: wip second draft of the PCB
Connections:
- net FAN_PWM: now also U1.63 (PC6); no longer U1.46 (PB10)
Changed lines of the file:
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@@
 	)
 	(no_connect
-		(at 116.84 133.35)
+		(at 116.84 100.33)
 	)
 	(no_connect
@@
 	(wire
 		(pts
+			(xy 116.84 133.35) (xy 121.92 133.35)
+		)
+		(stroke
+			(width 0)
+			(type default)
+		)
+	)
+	(wire
+		(pts
 			(xy 187.96 148.59) (xy 187.96 152.4)
 		)
@@
 	(wire
 		(pts
-			(xy 116.84 100.33) (xy 121.92 100.33)
-		)
-		(stroke
-			(width 0)
-			(type default)
-		)
-	)
-	(wire
-		(pts
 			(xy 34.29 182.88) (xy 34.29 184.15)
 		)
@@
 	(hierarchical_label "FAN_PWM"
 		(shape output)
-		(at 121.92 100.33 0)
+		(at 121.92 133.35 0)
 		(effects
 			(font

Commit message: third draft of the PCB
Connections:
- net OCP_V_N: now also U1.56 (PD9); no longer U1.55 (PD8)
- net OCP_V_P: now also U1.55 (PD8); no longer U1.88 (PD7)
- net OCP_W_N: now also U1.58 (PD11); no longer U1.57 (PD10)
- net OCP_W_P: now also U1.57 (PD10); no longer U1.56 (PD9)
- net IMU_INT2: now reaches U13.9 (INT2)
- net IMU_INT2: now also U1.93 (PB7)
- no-connect marks 32 -> 29
Changed lines of the file:
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@@
 	)
 	(no_connect
-		(at 55.88 57.15)
-	)
-	(no_connect
 		(at 116.84 54.61)
 	)
@@
 	)
 	(no_connect
-		(at 116.84 92.71)
-	)
-	(no_connect
-		(at 255.27 33.02)
-	)
-	(no_connect
 		(at 55.88 130.81)
 	)
@@
 	)
 	(no_connect
-		(at 55.88 125.73)
-	)
-	(no_connect
 		(at 255.27 85.09)
 	)
@@
 	)
 	(no_connect
+		(at 55.88 115.57)
+	)
+	(no_connect
 		(at 116.84 39.37)
 	)
@@
 	(wire
 		(pts
-			(xy 50.8 115.57) (xy 55.88 115.57)
+			(xy 46.99 153.67) (xy 46.99 154.94)
 		)
 		(stroke
@@
 	(wire
 		(pts
-			(xy 46.99 153.67) (xy 46.99 154.94)
+			(xy 160.02 78.74) (xy 160.02 80.01)
 		)
 		(stroke
@@
 	(wire
 		(pts
-			(xy 160.02 78.74) (xy 160.02 80.01)
+			(xy 116.84 92.71) (xy 121.92 92.71)
+		)
+		(stroke
+			(width 0)
+			(type default)
+		)
+	)
+	(wire
+		(pts
+			(xy 50.8 118.11) (xy 55.88 118.11)
 		)
 		(stroke
@@
 	(wire
 		(pts
-			(xy 50.8 118.11) (xy 55.88 118.11)
+			(xy 116.84 123.19) (xy 121.92 123.19)
 		)
 		(stroke
@@
 	(wire
 		(pts
-			(xy 116.84 123.19) (xy 121.92 123.19)
+			(xy 186.69 138.43) (xy 187.96 138.43)
 		)
 		(stroke
@@
 	(wire
 		(pts
-			(xy 186.69 138.43) (xy 187.96 138.43)
+			(xy 50.8 113.03) (xy 55.88 113.03)
 		)
 		(stroke
@@
 	(wire
 		(pts
-			(xy 50.8 113.03) (xy 55.88 113.03)
+			(xy 182.88 111.76) (xy 182.88 113.03)
 		)
 		(stroke
@@
 	(wire
 		(pts
-			(xy 182.88 111.76) (xy 182.88 113.03)
+			(xy 100.33 182.88) (xy 100.33 184.15)
 		)
 		(stroke
@@
 	(wire
 		(pts
-			(xy 100.33 182.88) (xy 100.33 184.15)
+			(xy 255.27 25.4) (xy 260.35 25.4)
 		)
 		(stroke
@@
 	(wire
 		(pts
-			(xy 255.27 25.4) (xy 260.35 25.4)
+			(xy 50.8 57.15) (xy 55.88 57.15)
 		)
 		(stroke
@@
 	(wire
 		(pts
+			(xy 50.8 125.73) (xy 55.88 125.73)
+		)
+		(stroke
+			(width 0)
+			(type default)
+		)
+	)
+	(wire
+		(pts
 			(xy 116.84 128.27) (xy 121.92 128.27)
 		)
@@
 	(wire
 		(pts
-			(xy 50.8 120.65) (xy 55.88 120.65)
-		)
-		(stroke
-			(width 0)
-			(type default)
-		)
-	)
-	(wire
-		(pts
 			(xy 22.86 31.75) (xy 55.88 31.75)
 		)
@@
 	(wire
 		(pts
-			(xy 64.77 182.88) (xy 64.77 184.15)
+			(xy 255.27 33.02) (xy 260.35 33.02)
 		)
 		(stroke
@@
 	(wire
 		(pts
-			(xy 34.29 53.34) (xy 34.29 49.53)
+			(xy 50.8 123.19) (xy 55.88 123.19)
 		)
 		(stroke
@@
 	(wire
 		(pts
-			(xy 116.84 77.47) (xy 121.92 77.47)
+			(xy 64.77 182.88) (xy 64.77 184.15)
 		)
 		(stroke
@@
 	(wire
 		(pts
-			(xy 166.37 25.4) (xy 173.99 25.4)
+			(xy 34.29 53.34) (xy 34.29 49.53)
 		)
 		(stroke
@@
 	(wire
 		(pts
-			(xy 49.53 184.15) (xy 57.15 184.15)
+			(xy 116.84 77.47) (xy 121.92 77.47)
 		)
 		(stroke
@@
 	(wire
 		(pts
-			(xy 19.05 46.99) (xy 19.05 53.34)
+			(xy 166.37 25.4) (xy 173.99 25.4)
 		)
 		(stroke
@@
 	(wire
 		(pts
-			(xy 158.75 35.56) (xy 158.75 36.83)
+			(xy 49.53 184.15) (xy 57.15 184.15)
 		)
 		(stroke
@@
 	(wire
 		(pts
-			(xy 35.56 153.67) (xy 35.56 154.94)
+			(xy 19.05 46.99) (xy 19.05 53.34)
 		)
 		(stroke
@@
 	(wire
 		(pts
-			(xy 50.8 123.19) (xy 55.88 123.19)
+			(xy 158.75 35.56) (xy 158.75 36.83)
+		)
+		(stroke
+			(width 0)
+			(type default)
+		)
+	)
+	(wire
+		(pts
+			(xy 35.56 153.67) (xy 35.56 154.94)
 		)
 		(stroke
@@
 	(wire
 		(pts
+			(xy 50.8 120.65) (xy 55.88 120.65)
+		)
+		(stroke
+			(width 0)
+			(type default)
+		)
+	)
+	(wire
+		(pts
 			(xy 27.94 63.5) (xy 34.29 63.5)
 		)
@@
 		)
 	)
+	(global_label "IMU_INT2"
+		(shape output)
+		(at 260.35 33.02 0)
+		(fields_autoplaced yes)
+		(effects
+			(font
+				(size 1.27 1.27)
+			)
+			(justify left)
+		)
+		(property "Intersheetrefs" "${INTERSHEET_REFS}"
+			(at 271.8019 33.02 0)
+			(effects
+				(font
+					(size 1.27 1.27)
+				)
+				(justify left)
+				(hide yes)
+			)
+		)
+	)
 	(global_label "IMU_INT1"
 		(shape input)
@@
 		)
 	)
+	(global_label "IMU_INT2"
+		(shape input)
+		(at 121.92 92.71 0)
+		(fields_autoplaced yes)
+		(effects
+			(font
+				(size 1.27 1.27)
+			)
+			(justify left)
+		)
+		(property "Intersheetrefs" "${INTERSHEET_REFS}"
+			(at 133.3719 92.71 0)
+			(effects
+				(font
+					(size 1.27 1.27)
+				)
+				(justify left)
+				(hide yes)
+			)
+		)
+	)
 	(global_label "SPI4_NSS"
 		(shape output)
@@
 	(hierarchical_label "OCP_V_N"
 		(shape input)
-		(at 50.8 118.11 180)
+		(at 50.8 120.65 180)
 		(effects
 			(font
@@
 	(hierarchical_label "OCP_V_P"
 		(shape input)
-		(at 50.8 115.57 180)
+		(at 50.8 118.11 180)
 		(effects
 			(font
@@
 	(hierarchical_label "OCP_W_P"
 		(shape input)
-		(at 50.8 120.65 180)
+		(at 50.8 123.19 180)
 		(effects
 			(font
@@
 	(hierarchical_label "OCP_W_N"
 		(shape input)
-		(at 50.8 123.19 180)
+		(at 50.8 125.73 180)
 		(effects
 			(font

Commit message: couple of ERC fixes
Parts:
- removed C94, C95: 1n, Capacitor_SMD:C_0201_0603Metric, symbol Device:C
Connections:
- no-connect marks 29 -> 30
