File: connectors.kicad_sch (KiCad schematic)
At the start: 35 parts, among them J10 Conn_01x06, J11 Conn_01x04, J12 USB4085-GF-A, J13 Conn_01x03, J14 Conn_01x03, J6 FTSH-107-01-L-DV-K-TR, J7 Conn_01x03, J8 Conn_01x02, J9 Conn_01x07, Q7 Si2302CDS

Commit message: WiP layout
Parts:
- removed C67, C68: 1u, Capacitor_SMD:C_0402_1005Metric, symbol Device:C
- removed J13: Conn_01x03, Connector_PinHeader_1.00mm:PinHeader_1x03_P1.00mm_Vertical, symbol Connector_Generic:Conn_01x03
- removed R39, R40: 0R, Resistor_SMD:R_0603_1608Metric, symbol Device:R
Connections:
- net GND: no longer D2.2 (GND)
- net USBVBUS: no longer names the net of J12.A4 (VBUS), J12.A9 (VBUS), J12.B4 (VBUS), J12.B9 (VBUS)
- net USBVBUS: no longer D2.5 (VBUS)
- no-connect marks 4 -> 7
Other:
- note removed: "Header for selecting +5V supply"
- note removed: "Header might be to weak for 3.5A"

Commit message: added the first draft of the layout
Parts:
- removed R30, R32: 10k, Resistor_SMD:R_0603_1608Metric, symbol Device:R
- added R11, R21: 10k, Resistor_SMD:R_0402_1005Metric, symbol Device:R
Connections:
- net EXT_TEMP1: now also R21.1
- net EXT_TEMP2: now also R11.1
- net GND: now also R11.2, R21.2
Changed lines of the file:
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@@
 	)
 	(symbol
-		(lib_id "Device:R")
-		(at 26.67 77.47 0)
-		(unit 1)
-		(exclude_from_sim no)
-		(in_bom yes)
-		(on_board yes)
-		(dnp no)
-		(fields_autoplaced yes)
-		(property "Reference" "R30"
-			(at 29.21 76.2 0)
-			(effects
-				(font
-					(size 1.27 1.27)
-				)
-				(justify left)
-			)
-		)
-		(property "Value" "10k"
-			(at 29.21 78.74 0)
-			(effects
-				(font
-					(size 1.27 1.27)
-				)
-				(justify left)
-			)
-		)
-		(property "Footprint" "Resistor_SMD:R_0603_1608Metric"
-			(at 24.892 77.47 90)
-			(effects
-				(font
-					(size 1.27 1.27)
-				)
-				(hide yes)
-			)
-		)
-		(property "Datasheet" "~"
-			(at 26.67 77.47 0)
-			(effects
-				(font
-					(size 1.27 1.27)
-				)
-				(hide yes)
-			)
-		)
-		(property "Description" "-55℃~+155℃ 100mW 10kΩ 75V Thick Film Resistor ±1% ±100ppm/℃ 0603 Chip Resistor - Surface Mount ROHS"
-			(at 26.67 77.47 0)
-			(effects
-				(font
-					(size 1.27 1.27)
-				)
-				(hide yes)
-			)
-		)
-		(property "LCSC" "C25804"
-			(at 26.67 77.47 0)
-			(effects
-				(font
-					(size 1.27 1.27)
-				)
-				(hide yes)
-			)
-		)
-		(pin "1"
-		)
-		(pin "2"
-		)
-		(instances
-			(project "NanoGaN"
-				(path "/aa8a494f-605e-4a00-9d3c-daec94709fcb/7b588d7e-2cba-479c-b934-83f1a7363076"
-					(reference "R30")
-					(unit 1)
-				)
-			)
-		)
-	)
-	(symbol
 		(lib_id "Power_Protection:USBLC6-2SC6")
 		(at 153.67 85.09 0)
@@
 	)
 	(symbol
+		(lib_id "Device:R")
+		(at 63.5 77.47 0)
+		(unit 1)
+		(exclude_from_sim no)
+		(in_bom yes)
+		(on_board yes)
+		(dnp no)
+		(property "Reference" "R21"
+			(at 65.532 77.47 90)
+			(effects
+				(font
+					(size 1.27 1.27)
+				)
+				(hide yes)
+			)
+		)
+		(property "Value" "10k"
+			(at 63.5 77.47 90)
+			(effects
+				(font
+					(size 1.27 1.27)
+				)
+			)
+		)
+		(property "Footprint" "Resistor_SMD:R_0402_1005Metric"
+			(at 61.722 77.47 90)
+			(effects
+				(font
+					(size 1.27 1.27)
+				)
+				(hide yes)
+			)
+		)
+		(property "Datasheet" "~"
+			(at 63.5 77.47 0)
+			(effects
+				(font
+					(size 1.27 1.27)
+				)
+				(hide yes)
+			)
+		)
+		(property "Description" "-55℃~+155℃ 10kΩ 50V 62.5mW Thick Film Resistor ±1% ±100ppm/℃ 0402 Chip Resistor - Surface Mount ROHS"
+			(at 63.5 77.47 0)
+			(effects
+				(font
+					(size 1.27 1.27)
+				)
+				(hide yes)
+			)
+		)
+		(property "LCSC" "C25744"
+			(at 63.5 77.47 0)
+			(effects
+				(font
+					(size 1.27 1.27)
+				)
+				(hide yes)
+			)
+		)
+		(pin "1"
+		)
+		(pin "2"
+		)
+		(instances
+			(project "NanoGaN"
+				(path "/aa8a494f-605e-4a00-9d3c-daec94709fcb/7b588d7e-2cba-479c-b934-83f1a7363076"
+					(reference "R21")
+					(unit 1)
+				)
+			)
+		)
+	)
+	(symbol
 		(lib_id "power:GND")
 		(at 118.11 35.56 0)
@@
 	)
 	(symbol
-		(lib_id "Device:R")
-		(at 63.5 77.47 0)
+		(lib_id "Device:C")
+		(at 55.88 161.29 0)
 		(unit 1)
 		(exclude_from_sim no)
@@
 		(on_board yes)
 		(dnp no)
-		(fields_autoplaced yes)
-		(property "Reference" "R32"
-			(at 66.04 76.2 0)
+		(property "Reference" "C60"
+			(at 58.42 160.02 0)
 			(effects
 				(font
@@
 				)
 				(justify left)
+				(hide yes)
 			)
 		)
-		(property "Value" "10k"
-			(at 66.04 78.74 0)
+		(property "Value" "4.7n"
+			(at 56.896 158.75 0)
 			(effects
 				(font
@@
 			)
 		)
-		(property "Footprint" "Resistor_SMD:R_0603_1608Metric"
-			(at 61.722 77.47 90)
+		(property "Footprint" "Capacitor_SMD:C_0402_1005Metric"
+			(at 56.8452 165.1 0)
 			(effects
 				(font
@@
 		)
 		(property "Datasheet" "~"
-			(at 63.5 77.47 0)
+			(at 55.88 161.29 0)
 			(effects
 				(font
@@
 			)
 		)
-		(property "Description" "-55℃~+155℃ 100mW 10kΩ 75V Thick Film Resistor ±1% ±100ppm/℃ 0603 Chip Resistor - Surface Mount ROHS"
-			(at 63.5 77.47 0)
+		(property "Description" "4.7nF 50V X7R ±10% 0402 Multilayer Ceramic Capacitors MLCC - SMD/SMT ROHS"
+			(at 55.88 161.29 0)
 			(effects
 				(font
@@
 			)
 		)
-		(property "LCSC" "C25804"
-			(at 63.5 77.47 0)
+		(property "LCSC" "C1538"
+			(at 55.88 161.29 0)
 			(effects
 				(font
@@
 			)
 		)
+		(property "Voltage Rating" "50V"
+			(at 58.674 163.83 0)
+			(effects
+				(font
+					(size 1.27 1.27)
+				)
+			)
+		)
 		(pin "1"
 		)
@@
 			(project "NanoGaN"
 				(path "/aa8a494f-605e-4a00-9d3c-daec94709fcb/7b588d7e-2cba-479c-b934-83f1a7363076"
-					(reference "R32")
+					(reference "C60")
 					(unit 1)
 				)
@@
 	)
 	(symbol
-		(lib_id "Device:C")
-		(at 55.88 161.29 0)
+		(lib_id "Connector_Generic:Conn_01x02")
+		(at 111.76 137.16 0)
+		(mirror y)
 		(unit 1)
 		(exclude_from_sim no)
@@
 		(on_board yes)
 		(dnp no)
-		(property "Reference" "C60"
-			(at 58.42 160.02 0)
-			(effects
-				(font
-					(size 1.27 1.27)
-				)
-				(justify left)
-				(hide yes)
-			)
-		)
-		(property "Value" "4.7n"
-			(at 56.896 158.75 0)
+		(property "Reference" "J8"
+			(at 107.95 137.922 0)
 			(effects
 				(font
 					(size 1.27 1.27)
 				)
-				(justify left)
 			)
 		)
-		(property "Footprint" "Capacitor_SMD:C_0402_1005Metric"
-			(at 56.8452 165.1 0)
+		(property "Value" "Conn_01x02"
+			(at 101.092 139.446 0)
 			(effects
 				(font
@@
 			)
 		)
-		(property "Datasheet" "~"
-			(at 55.88 161.29 0)
+		(property "Footprint" "Connector_JST:JST_EH_B2B-EH-A_1x02_P2.50mm_Vertical"
+			(at 111.76 137.16 0)
 			(effects
 				(font
@@
 			)
 		)
-		(property "Description" "4.7nF 50V X7R ±10% 0402 Multilayer Ceramic Capacitors MLCC - SMD/SMT ROHS"
-			(at 55.88 161.29 0)
+		(property "Datasheet" "~"
+			(at 111.76 137.16 0)
 			(effects
 				(font
@@
 			)
 		)
-		(property "LCSC" "C1538"
-			(at 55.88 161.29 0)
+		(property "Description" "Generic connector, single row, 01x02, script generated (kicad-library-utils/schlib/autogen/connector/)"
+			(at 111.76 137.16 0)
 			(effects
 				(font
@@
 			)
 		)
-		(property "Voltage Rating" "50V"
-			(at 58.674 163.83 0)
-			(effects
-				(font
-					(size 1.27 1.27)
-				)
-			)
+		(pin "2"
 		)
 		(pin "1"
 		)
-		(pin "2"
-		)
 		(instances
-			(project "NanoGaN"
+			(project ""
 				(path "/aa8a494f-605e-4a00-9d3c-daec94709fcb/7b588d7e-2cba-479c-b934-83f1a7363076"
-					(reference "C60")
+					(reference "J8")
 					(unit 1)
 				)
@@
 	)
 	(symbol
-		(lib_id "Connector_Generic:Conn_01x02")
-		(at 111.76 137.16 0)
-		(mirror y)
+		(lib_id "Device:R")
+		(at 26.67 77.47 0)
 		(unit 1)
 		(exclude_from_sim no)
@@
 		(on_board yes)
 		(dnp no)
-		(property "Reference" "J8"
-			(at 107.95 137.922 0)
+		(property "Reference" "R11"
+			(at 28.702 77.47 90)
 			(effects
 				(font
 					(size 1.27 1.27)
 				)
+				(hide yes)
 			)
 		)
-		(property "Value" "Conn_01x02"
-			(at 101.092 139.446 0)
+		(property "Value" "10k"
+			(at 26.67 77.47 90)
 			(effects
 				(font
 					(size 1.27 1.27)
 				)
-				(hide yes)
 			)
 		)
-		(property "Footprint" "Connector_JST:JST_EH_B2B-EH-A_1x02_P2.50mm_Vertical"
-			(at 111.76 137.16 0)
+		(property "Footprint" "Resistor_SMD:R_0402_1005Metric"
+			(at 24.892 77.47 90)
 			(effects
 				(font
@@
 		)
 		(property "Datasheet" "~"
-			(at 111.76 137.16 0)
+			(at 26.67 77.47 0)
 			(effects
 				(font
@@
 			)
 		)
-		(property "Description" "Generic connector, single row, 01x02, script generated (kicad-library-utils/schlib/autogen/connector/)"
-			(at 111.76 137.16 0)
+		(property "Description" "-55℃~+155℃ 10kΩ 50V 62.5mW Thick Film Resistor ±1% ±100ppm/℃ 0402 Chip Resistor - Surface Mount ROHS"
+			(at 26.67 77.47 0)
 			(effects
 				(font
@@
 			)
 		)
-		(pin "2"
+		(property "LCSC" "C25744"
+			(at 26.67 77.47 0)
+			(effects
+				(font
+					(size 1.27 1.27)
+				)
+				(hide yes)
+			)
 		)
 		(pin "1"
 		)
+		(pin "2"
+		)
 		(instances
-			(project ""
+			(project "NanoGaN"
 				(path "/aa8a494f-605e-4a00-9d3c-daec94709fcb/7b588d7e-2cba-479c-b934-83f1a7363076"
-					(reference "J8")
+					(reference "R11")
 					(unit 1)
 				)

Commit message: wip layout
Parts:
- removed J12: USB4085-GF-A, Connector_USB:USB_C_Receptacle_GCT_USB4085, symbol NanoGaN:USB_C_Receptacle_USB2.0_14P
- added J12: USB_C_Receptacle_USB2.0_16P, Connector_USB:USB_C_Receptacle_GCT_USB4105-xx-A_16P_TopMnt_Horizontal, symbol Connector:USB_C_Receptacle_USB2.0_16P
Connections:
- net D+: now also J12.A6 (D+), J12.B6 (D+)
- net D-: now also J12.A7 (D-), J12.B7 (D-)
- net GND: now also J12.A1 (GND), J12.A12 (GND), J12.B1 (GND), J12.B12 (GND), J12.S1 (SHIELD)
- net USBCC1: now also J12.A5 (CC1)
- net USBCC2: now also J12.B5 (CC2)
- new net: J12.A4 (VBUS), J12.A9 (VBUS), J12.B4 (VBUS), J12.B9 (VBUS)
- no-connect marks 7 -> 9
Changed lines of the file:
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@@
 		(at 153.67 92.71)
+	)
+	(no_connect
+		(at 130.81 100.33)
+	)
+	(no_connect
+		(at 130.81 97.79)
 	)
 	(wire
@@
 			)
 			(justify left)
+		)
+	)
+	(symbol
+		(lib_id "Connector:USB_C_Receptacle_USB2.0_16P")
+		(at 115.57 85.09 0)
+		(unit 1)
+		(exclude_from_sim no)
+		(in_bom yes)
+		(on_board yes)
+		(dnp no)
+		(property "Reference" "J12"
+			(at 106.934 66.04 0)
+			(effects
+				(font
+					(size 1.27 1.27)
+				)
+			)
+		)
+		(property "Value" "USB_C_Receptacle_USB2.0_16P"
+			(at 115.57 64.77 0)
+			(effects
+				(font
+					(size 1.27 1.27)
+				)
+				(hide yes)
+			)
+		)
+		(property "Footprint" "Connector_USB:USB_C_Receptacle_GCT_USB4105-xx-A_16P_TopMnt_Horizontal"
+			(at 174.244 115.316 0)
+			(effects
+				(font
+					(size 1.27 1.27)
+				)
+				(hide yes)
+			)
+		)
+		(property "Datasheet" "https://www.usb.org/sites/default/files/documents/usb_type-c.zip"
+			(at 119.38 85.09 0)
+			(effects
+				(font
+					(size 1.27 1.27)
+				)
+				(hide yes)
+			)
+		)
+		(property "Description" "USB 2.0-only 16P Type-C Receptacle connector"
+			(at 115.57 85.09 0)
+			(effects
+				(font
+					(size 1.27 1.27)
+				)
+				(hide yes)
+			)
+		)
+		(property "LCSC" "C2988369"
+			(at 115.57 85.09 0)
+			(effects
+				(font
+					(size 1.27 1.27)
+				)
+				(hide yes)
+			)
+		)
+		(pin "B8"
+		)
+		(pin "A5"
+		)
+		(pin "A8"
+		)
+		(pin "A9"
+		)
+		(pin "B6"
+		)
+		(pin "A6"
+		)
+		(pin "A7"
+		)
+		(pin "A12"
+		)
+		(pin "B9"
+		)
+		(pin "B1"
+		)
+		(pin "A1"
+		)
+		(pin "S1"
+		)
+		(pin "A4"
+		)
+		(pin "B5"
+		)
+		(pin "B4"
+		)
+		(pin "B7"
+		)
+		(pin "B12"
+		)
+		(instances
+			(project ""
+				(path "/aa8a494f-605e-4a00-9d3c-daec94709fcb/7b588d7e-2cba-479c-b934-83f1a7363076"
+					(reference "J12")
+					(unit 1)
+				)
+			)
 		)
 	)
@@
 					(unit 1)
 				)
-			)
-		)
-	)
-	(symbol
-		(lib_id "NanoGaN:USB_C_Receptacle_USB2.0_14P")
-		(at 115.57 85.09 0)
-		(unit 1)
-		(exclude_from_sim no)
-		(in_bom yes)
-		(on_board yes)
-		(dnp no)
-		(property "Reference" "J12"
-			(at 106.934 66.294 0)
-			(effects
-				(font
-					(size 1.27 1.27)
-				)
-			)
-		)
-		(property "Value" "USB4085-GF-A"
-			(at 124.46 104.394 0)
-			(effects
-				(font
-					(size 1.27 1.27)
-				)
-			)
-		)
-		(property "Footprint" "Connector_USB:USB_C_Receptacle_GCT_USB4085"
-			(at 119.38 85.09 0)
-			(effects
-				(font
-					(size 1.27 1.27)
-				)
-				(hide yes)
-			)
-		)
-		(property "Datasheet" "https://www.usb.org/sites/default/files/documents/usb_type-c.zip"
-			(at 119.38 85.09 0)
-			(effects
-				(font
-					(size 1.27 1.27)
-				)
-				(hide yes)
-			)
-		)
-		(property "Description" "USB 2.0-only 14P Type-C Receptacle connector"
-			(at 115.57 85.09 0)
-			(effects
-				(font
-					(size 1.27 1.27)
-				)
-				(hide yes)
-			)
-		)
-		(pin "A9"
-		)
-		(pin "S1"
-		)
-		(pin "B1"
-		)
-		(pin "A8"
-		)
-		(pin "A1"
-		)
-		(pin "B8"
-		)
-		(pin "A4"
-		)
-		(pin "B7"
-		)
-		(pin "A12"
-		)
-		(pin "B12"
-		)
-		(pin "B4"
-		)
-		(pin "A7"
-		)
-		(pin "B6"
-		)
-		(pin "B9"
-		)
-		(pin "A5"
-		)
-		(pin "B5"
-		)
-		(pin "A6"
-		)
-		(instances
-			(project ""
-				(path "/aa8a494f-605e-4a00-9d3c-daec94709fcb/7b588d7e-2cba-479c-b934-83f1a7363076"
-					(reference "J12")
-					(unit 1)
-				)

Commit message: first draft of the PCB
Connections:
- net +5V: now also D2.5 (VBUS)
- net GND: now also D2.2 (GND)
- no-connect marks 9 -> 7
Changed lines of the file:
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@@
 	)
 	(no_connect
-		(at 153.67 80.01)
-	)
-	(no_connect
 		(at 52.07 33.02)
 	)
@@
 	)
 	(no_connect
-		(at 153.67 92.71)
-	)
-	(no_connect
 		(at 130.81 100.33)
 	)
@@
 	(wire
 		(pts
+			(xy 153.67 93.98) (xy 153.67 92.71)
+		)
+		(stroke
+			(width 0)
+			(type default)
+		)
+	)
+	(wire
+		(pts
 			(xy 38.1 135.89) (xy 44.45 135.89)
 		)
@@
 	(wire
 		(pts
+			(xy 153.67 77.47) (xy 153.67 80.01)
+		)
+		(stroke
+			(width 0)
+			(type default)
+		)
+	)
+	(wire
+		(pts
 			(xy 71.12 149.86) (xy 71.12 157.48)
 		)
@@
 	)
 	(symbol
+		(lib_id "power:GND")
+		(at 115.57 113.03 0)
+		(unit 1)
+		(exclude_from_sim no)
+		(in_bom yes)
+		(on_board yes)
+		(dnp no)
+		(property "Reference" "#PWR080"
+			(at 115.57 119.38 0)
+			(effects
+				(font
+					(size 1.27 1.27)
+				)
+				(hide yes)
+			)
+		)
+		(property "Value" "GND"
+			(at 115.57 117.094 0)
+			(effects
+				(font
+					(size 1.27 1.27)
+				)
+			)
+		)
+		(property "Footprint" ""
+			(at 115.57 113.03 0)
+			(effects
+				(font
+					(size 1.27 1.27)
+				)
+				(hide yes)
+			)
+		)
+		(property "Datasheet" ""
+			(at 115.57 113.03 0)
+			(effects
+				(font
+					(size 1.27 1.27)
+				)
+				(hide yes)
+			)
+		)
+		(property "Description" ""
+			(at 115.57 113.03 0)
+			(effects
+				(font
+					(size 1.27 1.27)
+				)
+			)
+		)
+		(pin "1"
+		)
+		(instances
+			(project "NanoGaN"
+				(path "/aa8a494f-605e-4a00-9d3c-daec94709fcb/7b588d7e-2cba-479c-b934-83f1a7363076"
+					(reference "#PWR080")
+					(unit 1)
+				)
+			)
+		)
+	)
+	(symbol
 		(lib_id "Device:D_Schottky")
 		(at 127 140.97 270)
@@
 		)
 		(property "Value" "USBLC6-2SC6"
-			(at 160.782 93.218 0)
+			(at 169.672 92.202 0)
 			(effects
 				(font
@@
 	)
 	(symbol
+		(lib_id "power:+3.3V")
+		(at 153.67 77.47 0)
+		(unit 1)
+		(exclude_from_sim no)
+		(in_bom yes)
+		(on_board yes)
+		(dnp no)
+		(property "Reference" "#PWR0113"
+			(at 153.67 81.28 0)
+			(effects
+				(font
+					(size 1.27 1.27)
+				)
+				(hide yes)
+			)
+		)
+		(property "Value" "+5V"
+			(at 153.67 73.914 0)
+			(effects
+				(font
+					(size 1.27 1.27)
+				)
+			)
+		)
+		(property "Footprint" ""
+			(at 153.67 77.47 0)
+			(effects
+				(font
+					(size 1.27 1.27)
+				)
+				(hide yes)
+			)
+		)
+		(property "Datasheet" ""
+			(at 153.67 77.47 0)
+			(effects
+				(font
+					(size 1.27 1.27)
+				)
+				(hide yes)
+			)
+		)
+		(property "Description" ""
+			(at 153.67 77.47 0)
+			(effects
+				(font
+					(size 1.27 1.27)
+				)
+			)
+		)
+		(pin "1"
+		)
+		(instances
+			(project "NanoGaN"
+				(path "/aa8a494f-605e-4a00-9d3c-daec94709fcb/7b588d7e-2cba-479c-b934-83f1a7363076"
+					(reference "#PWR0113")
+					(unit 1)
+				)
+			)
+		)
+	)
+	(symbol
 		(lib_id "power:+5V")
 		(at 119.38 135.89 0)
@@
 	)
 	(symbol
-		(lib_id "power:GND")
-		(at 115.57 113.03 0)
-		(unit 1)
-		(exclude_from_sim no)
-		(in_bom yes)
-		(on_board yes)
-		(dnp no)
-		(property "Reference" "#PWR0109"
-			(at 115.57 119.38 0)
-			(effects
-				(font
-					(size 1.27 1.27)
-				)
-				(hide yes)
-			)
-		)
-		(property "Value" "GND"
-			(at 115.57 117.094 0)
-			(effects
-				(font
-					(size 1.27 1.27)
-				)
-			)
-		)
-		(property "Footprint" ""
-			(at 115.57 113.03 0)
-			(effects
-				(font
-					(size 1.27 1.27)
-				)
-				(hide yes)
-			)
-		)
-		(property "Datasheet" ""
-			(at 115.57 113.03 0)
-			(effects
-				(font
-					(size 1.27 1.27)
-				)
-				(hide yes)
-			)
-		)
-		(property "Description" ""
-			(at 115.57 113.03 0)
-			(effects
-				(font
-					(size 1.27 1.27)
-				)
-			)
-		)
-		(pin "1"
-		)
-		(instances
-			(project "NanoGaN"
-				(path "/aa8a494f-605e-4a00-9d3c-daec94709fcb/7b588d7e-2cba-479c-b934-83f1a7363076"
-					(reference "#PWR0109")
-					(unit 1)
-				)
-			)
-		)
-	)
-	(symbol
 		(lib_id "Connector_Generic:Conn_01x06")
 		(at 22.86 149.86 0)
@@
 					(unit 1)
 				)
+			)
+		)
+	)
+	(symbol
+		(lib_id "power:GND")
+		(at 153.67 93.98 0)
+		(unit 1)
+		(exclude_from_sim no)
+		(in_bom yes)
+		(on_board yes)
+		(dnp no)
+		(property "Reference" "#PWR0109"
+			(at 153.67 100.33 0)
+			(effects
+				(font
+					(size 1.27 1.27)
+				)
+				(hide yes)
+			)
+		)
+		(property "Value" "GND"
+			(at 153.67 98.044 0)
+			(effects
+				(font
+					(size 1.27 1.27)
+				)
+			)
+		)
+		(property "Footprint" ""
+			(at 153.67 93.98 0)
+			(effects
+				(font
+					(size 1.27 1.27)
+				)
+				(hide yes)
+			)
+		)
+		(property "Datasheet" ""
+			(at 153.67 93.98 0)
+			(effects
+				(font
+					(size 1.27 1.27)
+				)
+				(hide yes)
+			)
+		)
+		(property "Description" ""
+			(at 153.67 93.98 0)
+			(effects
+				(font
+					(size 1.27 1.27)
+				)
+			)
+		)
+		(pin "1"
+		)
+		(instances
+			(project "NanoGaN"
+				(path "/aa8a494f-605e-4a00-9d3c-daec94709fcb/7b588d7e-2cba-479c-b934-83f1a7363076"
+					(reference "#PWR0109")
+					(unit 1)
+				)

Commit message: wip second draft of the PCB
Parts:
- removed R50: 100, Resistor_SMD:R_0402_1005Metric, symbol Device:R
- added C93: 4u7, Capacitor_SMD:C_0402_1005Metric, symbol Device:C
- added Q8: AO3400A, NanoGaN:SOT-23_3, symbol Simulation_SPICE:NMOS
- added R39: 0402WGF1000TCE, Resistor_SMD:R_0402_1005Metric, symbol Device:R
- added R40: 0402WGF1001TCE, Resistor_SMD:R_0402_1005Metric, symbol NanoGaN:R
- Q7: value Si2302CDS -> AO3400A; footprint NanoGaN:SOT-23_Si2302CDS -> NanoGaN:SOT-23_3; LCSC C10488 -> (none)
- R42: value 10k -> 0402WGF1002TCE; Resistance (none) -> 10k
- R43: value 100 -> 0402WGF2200TCE; LCSC C25076 -> C25091; Resistance (none) -> 220
Connections:
- net +5V: now also C93.1, R40.1
- net FANN: now also C93.2
- net GND: now also R42.2, Q8.3 (S); no longer R42.1
- net SERVO: now also R39.2
- net SERVO_IN: now also R39.1
- removed net FAN_Q_GATE: Q7.2 (G), R42.2, R43.1
- new net FAN_GATE: Q7.2 (G), Q8.1 (D), R40.2
- new net FAN_GATE_B: Q8.2 (G), R42.1, R43.1
Other:
- note added: "Differential Pair settings"
- note added: "tau = R*C = 1k * 630pf = 630ns"
- note added: "tau = R*C = 220 * 630pf = 138ns"
- moved on the sheet: D3, J11, J8, R43
