File: power.kicad_sch (KiCad schematic)
At the start: 37 parts, among them U2 LMR51635XDDCR, U3 AMS1117

Commit message: wip layout
Parts:
- removed NT1, NT2: NetTie_2, NetTie:NetTie-2_SMD_Pad0.5mm, symbol Device:NetTie_2
- C18: footprint Capacitor_SMD:C_0402_1005Metric -> Capacitor_SMD:C_0603_1608Metric_Pad1.08x0.95mm_HandSolder
Connections:
- net AGND is gone; now on net GND: C10.2, C9.2
- net PGND is gone; now on net GND: C1.2, C11.2, C12.2, C13.2, C14.2, C18.2, C2.2, C27.2, C3.2, C35.2, C4.2, C6.2, C68.2, C7.2, C81.2, C82.2, C86.2, C88.2, C90.2, R2.2, R5.2, U2.4 (GND)
Changed lines of the file:
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@@
 	(wire
 		(pts
-			(xy 49.53 93.98) (xy 57.15 93.98)
-		)
-		(stroke
-			(width 0)
-			(type default)
-		)
-	)
-	(wire
-		(pts
 			(xy 63.5 125.73) (xy 63.5 129.54)
 		)
@@
 	(wire
 		(pts
-			(xy 38.1 93.98) (xy 44.45 93.98)
+			(xy 38.1 93.98) (xy 57.15 93.98)
 		)
 		(stroke
@@
 	(wire
 		(pts
-			(xy 107.95 93.98) (xy 114.3 93.98)
-		)
-		(stroke
-			(width 0)
-			(type default)
-		)
-	)
-	(wire
-		(pts
 			(xy 127 139.7) (xy 135.89 139.7)
 		)
@@
 	(wire
 		(pts
-			(xy 96.52 93.98) (xy 102.87 93.98)
+			(xy 96.52 93.98) (xy 114.3 93.98)
 		)
 		(stroke
@@
 			)
 		)
-		(property "Value" "AGND"
+		(property "Value" "GND"
 			(at 125.73 100.584 0)
 			(effects
@@
 	)
 	(symbol
-		(lib_id "Device:NetTie_2")
-		(at 105.41 93.98 0)
-		(unit 1)
-		(exclude_from_sim no)
-		(in_bom no)
-		(on_board yes)
-		(dnp no)
-		(property "Reference" "NT2"
-			(at 105.664 92.964 0)
-			(effects
-				(font
-					(size 1.27 1.27)
-				)
-			)
-		)
-		(property "Value" "NetTie_2"
-			(at 105.41 91.44 0)
-			(effects
-				(font
-					(size 1.27 1.27)
-				)
-				(hide yes)
-			)
-		)
-		(property "Footprint" "NetTie:NetTie-2_SMD_Pad0.5mm"
-			(at 105.41 93.98 0)
-			(effects
-				(font
-					(size 1.27 1.27)
-				)
-				(hide yes)
-			)
-		)
-		(property "Datasheet" "~"
-			(at 105.41 93.98 0)
-			(effects
-				(font
-					(size 1.27 1.27)
-				)
-				(hide yes)
-			)
-		)
-		(property "Description" "Net tie, 2 pins"
-			(at 105.41 93.98 0)
-			(effects
-				(font
-					(size 1.27 1.27)
-				)
-				(hide yes)
-			)
-		)
-		(pin "2"
-		)
-		(pin "1"
-		)
-		(instances
-			(project "NanoGaN"
-				(path "/aa8a494f-605e-4a00-9d3c-daec94709fcb/2aff88eb-0d92-4253-8876-ba05112be4d6"
-					(reference "NT2")
-					(unit 1)
-				)
-			)
-		)
-	)
-	(symbol
 		(lib_id "Device:R_Small")
 		(at 96.52 90.17 180)
@@
 			)
 		)
-		(property "Footprint" "Capacitor_SMD:C_0402_1005Metric"
+		(property "Footprint" "Capacitor_SMD:C_0603_1608Metric_Pad1.08x0.95mm_HandSolder"
 			(at 50.4952 184.15 0)
 			(effects
@@
 			)
 		)
-		(property "LCSC" ""
-			(at 49.53 180.34 0)
-			(effects
-				(font
-					(size 1.27 1.27)
-				)
-				(hide yes)
-			)
-		)
 		(property "Voltage Rating" "6.3V"
 			(at 52.324 182.88 0)
@@
 					(unit 1)
 				)
-			)
-		)
-	)
-	(symbol
-		(lib_id "Device:NetTie_2")
-		(at 46.99 93.98 0)
-		(unit 1)
-		(exclude_from_sim no)
-		(in_bom no)
-		(on_board yes)
-		(dnp no)
-		(property "Reference" "NT1"
-			(at 47.244 92.964 0)
-			(effects
-				(font
-					(size 1.27 1.27)
-				)
-			)
-		)
-		(property "Value" "NetTie_2"
-			(at 46.99 91.44 0)
-			(effects
-				(font
-					(size 1.27 1.27)
-				)
-				(hide yes)
-			)
-		)
-		(property "Footprint" "NetTie:NetTie-2_SMD_Pad0.5mm"
-			(at 46.99 93.98 0)
-			(effects
-				(font
-					(size 1.27 1.27)
-				)
-				(hide yes)
-			)
-		)
-		(property "Datasheet" "~"
-			(at 46.99 93.98 0)
-			(effects
-				(font
-					(size 1.27 1.27)
-				)
-				(hide yes)
-			)
-		)
-		(property "Description" "Net tie, 2 pins"
-			(at 46.99 93.98 0)
-			(effects
-				(font
-					(size 1.27 1.27)
-				)
-				(hide yes)
-			)
-		)
-		(pin "2"
-		)
-		(pin "1"
-		)
-		(instances
-			(project "NanoGaN"
-				(path "/aa8a494f-605e-4a00-9d3c-daec94709fcb/2aff88eb-0d92-4253-8876-ba05112be4d6"
-					(reference "NT1")
-					(unit 1)
-				)

Commit message: wip layout
Parts:
- added C79: 4u7, Capacitor_SMD:C_0402_1005Metric, symbol Device:C
Connections:
- net +5V: now also C79.1
- net GND: now also C79.2
Changed lines of the file:
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@@
 	)
 	(junction
+		(at 38.1 93.98)
+		(diameter 0)
+		(color 0 0 0 0)
+	)
+	(junction
 		(at 88.9 93.98)
 		(diameter 0)
@@
 	)
 	(junction
+		(at 38.1 81.28)
+		(diameter 0)
+		(color 0 0 0 0)
+	)
+	(junction
 		(at 120.65 35.56)
 		(diameter 0)
@@
 	)
 	(junction
-		(at 38.1 81.28)
+		(at 45.72 81.28)
 		(diameter 0)
 		(color 0 0 0 0)
@@
 	)
 	(junction
-		(at 38.1 93.98)
+		(at 45.72 93.98)
 		(diameter 0)
 		(color 0 0 0 0)
@@
 	(wire
 		(pts
-			(xy 38.1 91.44) (xy 38.1 93.98)
+			(xy 45.72 91.44) (xy 45.72 93.98)
+		)
+		(stroke
+			(width 0)
+			(type default)
+		)
+	)
+	(wire
+		(pts
+			(xy 38.1 81.28) (xy 45.72 81.28)
 		)
 		(stroke
@@
 	(wire
 		(pts
+			(xy 57.15 93.98) (xy 73.66 93.98)
+		)
+		(stroke
+			(width 0)
+			(type default)
+		)
+	)
+	(wire
+		(pts
 			(xy 144.78 129.54) (xy 144.78 125.73)
 		)
@@
 	(wire
 		(pts
-			(xy 57.15 93.98) (xy 73.66 93.98)
+			(xy 45.72 93.98) (xy 57.15 93.98)
 		)
 		(stroke
@@
 	(wire
 		(pts
-			(xy 38.1 93.98) (xy 57.15 93.98)
+			(xy 63.5 139.7) (xy 76.2 139.7)
 		)
 		(stroke
@@
 	(wire
 		(pts
-			(xy 63.5 139.7) (xy 76.2 139.7)
+			(xy 135.89 137.16) (xy 135.89 139.7)
 		)
 		(stroke
@@
 	(wire
 		(pts
-			(xy 135.89 137.16) (xy 135.89 139.7)
+			(xy 128.27 91.44) (xy 128.27 93.98)
 		)
 		(stroke
@@
 	(wire
 		(pts
-			(xy 128.27 91.44) (xy 128.27 93.98)
+			(xy 100.33 125.73) (xy 88.9 125.73)
 		)
 		(stroke
@@
 	(wire
 		(pts
-			(xy 100.33 125.73) (xy 88.9 125.73)
+			(xy 38.1 93.98) (xy 38.1 91.44)
 		)
 		(stroke
@@
 	(wire
 		(pts
-			(xy 38.1 83.82) (xy 38.1 81.28)
+			(xy 45.72 83.82) (xy 45.72 81.28)
 		)
 		(stroke
@@
 	(wire
 		(pts
-			(xy 38.1 81.28) (xy 49.53 81.28)
+			(xy 45.72 81.28) (xy 49.53 81.28)
 		)
 		(stroke
@@
 	(wire
 		(pts
+			(xy 38.1 83.82) (xy 38.1 81.28)
+		)
+		(stroke
+			(width 0)
+			(type default)
+		)
+	)
+	(wire
+		(pts
 			(xy 19.05 35.56) (xy 19.05 33.02)
 		)
@@
 	(wire
 		(pts
+			(xy 45.72 93.98) (xy 38.1 93.98)
+		)
+		(stroke
+			(width 0)
+			(type default)
+		)
+	)
+	(wire
+		(pts
 			(xy 27.94 33.02) (xy 36.83 33.02)
 		)
@@
 	)
 	(symbol
+		(lib_id "Device:C")
+		(at 38.1 87.63 0)
+		(unit 1)
+		(exclude_from_sim no)
+		(in_bom yes)
+		(on_board yes)
+		(dnp no)
+		(property "Reference" "C79"
+			(at 40.64 86.36 0)
+			(effects
+				(font
+					(size 1.27 1.27)
+				)
+				(justify left)
+				(hide yes)
+			)
+		)
+		(property "Value" "4u7"
+			(at 39.116 85.09 0)
+			(effects
+				(font
+					(size 1.27 1.27)
+				)
+				(justify left)
+			)
+		)
+		(property "Footprint" "Capacitor_SMD:C_0402_1005Metric"
+			(at 39.0652 91.44 0)
+			(effects
+				(font
+					(size 1.27 1.27)
+				)
+				(hide yes)
+			)
+		)
+		(property "Datasheet" "~"
+			(at 38.1 87.63 0)
+			(effects
+				(font
+					(size 1.27 1.27)
+				)
+				(hide yes)
+			)
+		)
+		(property "Description" "10V 4.7uF X5R ±20% 0402 Multilayer Ceramic Capacitors MLCC - SMD/SMT ROHS"
+			(at 38.1 87.63 0)
+			(effects
+				(font
+					(size 1.27 1.27)
+				)
+				(hide yes)
+			)
+		)
+		(property "LCSC" "C23733"
+			(at 38.1 87.63 0)
+			(effects
+				(font
+					(size 1.27 1.27)
+				)
+				(hide yes)
+			)
+		)
+		(property "Voltage Rating" "10V"
+			(at 40.894 90.17 0)
+			(effects
+				(font
+					(size 1.27 1.27)
+				)
+			)
+		)
+		(pin "1"
+		)
+		(pin "2"
+		)
+		(instances
+			(project "NanoGaN"
+				(path "/aa8a494f-605e-4a00-9d3c-daec94709fcb/2aff88eb-0d92-4253-8876-ba05112be4d6"
+					(reference "C79")
+					(unit 1)
+				)
+			)
+		)
+	)
+	(symbol
 		(lib_id "power:GND")
 		(at 120.65 44.45 0)
@@
 	(symbol
 		(lib_id "Device:C")
-		(at 38.1 87.63 0)
+		(at 45.72 87.63 0)
 		(unit 1)
 		(exclude_from_sim no)
@@
 		(dnp no)
 		(property "Reference" "C7"
-			(at 40.64 86.36 0)
+			(at 48.26 86.36 0)
 			(effects
 				(font
@@
 		)
 		(property "Value" "4u7"
-			(at 39.116 85.09 0)
+			(at 46.736 85.09 0)
 			(effects
 				(font
@@
 		)
 		(property "Footprint" "Capacitor_SMD:C_0402_1005Metric"
-			(at 39.0652 91.44 0)
+			(at 46.6852 91.44 0)
 			(effects
 				(font
@@
 		)
 		(property "Datasheet" "~"
-			(at 38.1 87.63 0)
+			(at 45.72 87.63 0)
 			(effects
 				(font
@@
 		)
 		(property "Description" "10V 4.7uF X5R ±20% 0402 Multilayer Ceramic Capacitors MLCC - SMD/SMT ROHS"
-			(at 38.1 87.63 0)
+			(at 45.72 87.63 0)
 			(effects
 				(font
@@
 		)
 		(property "LCSC" "C23733"
-			(at 38.1 87.63 0)
+			(at 45.72 87.63 0)
 			(effects
 				(font
@@
 		)
 		(property "Voltage Rating" "10V"
-			(at 40.894 90.17 0)
+			(at 48.514 90.17 0)
 			(effects
 				(font

Commit message: wip second draft of the PCB
Parts:
- added R7: 0402WGF0000TCE, Resistor_SMD:R_0402_1005Metric, symbol NanoGaN:R
Connections:
- net U_DC_SENS: now also R7.2; no longer C18.1, R4.2, R5.1
- new net: C18.1, R4.2, R5.1, R7.1
Other:
- note added: "Extra ceramic (X7R) capacitors for improving switching performance."
- note removed: "Extra capacitors for improving switching performance."
Changed lines of the file:
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@@
 		)
 	)
-	(text "Extra capacitors for improving switching performance."
+	(text "Extra ceramic (X7R) capacitors \nfor improving switching performance."
 		(exclude_from_sim no)
-		(at 125.222 149.098 0)
+		(at 130.81 149.352 0)
 		(effects
 			(font
@@
 	(wire
 		(pts
-			(xy 49.53 173.99) (xy 55.88 173.99)
+			(xy 49.53 173.99) (xy 58.42 173.99)
 		)
 		(stroke
@@
 	(wire
 		(pts
+			(xy 66.04 173.99) (xy 71.12 173.99)
+		)
+		(stroke
+			(width 0)
+			(type default)
+		)
+	)
+	(wire
+		(pts
 			(xy 38.1 139.7) (xy 38.1 142.24)
 		)
@@
 	(hierarchical_label "U_DC_SENS"
 		(shape input)
-		(at 55.88 173.99 0)
+		(at 71.12 173.99 0)
 		(effects
 			(font
@@
 					(unit 1)
 				)
+			)
+		)
+	)
+	(symbol
+		(lib_id "NanoGaN:R")
+		(at 62.23 173.99 90)
+		(unit 1)
+		(exclude_from_sim no)
+		(in_bom yes)
+		(on_board yes)
+		(dnp no)
+		(property "Reference" "R7"
+			(at 62.23 171.958 90)
+			(effects
+				(font
+					(size 1.27 1.27)
+				)
+			)
+		)
+		(property "Value" "0402WGF0000TCE"
+			(at 62.23 170.18 90)
+			(effects
+				(font
+					(size 1.27 1.27)
+				)
+				(hide yes)
+			)
+		)
+		(property "Footprint" "Resistor_SMD:R_0402_1005Metric"
+			(at 62.23 175.768 90)
+			(effects
+				(font
+					(size 1.27 1.27)
+				)
+				(hide yes)
+			)
+		)
+		(property "Datasheet" "~"
+			(at 62.23 173.99 0)
+			(effects
+				(font
+					(size 1.27 1.27)
+				)
+				(hide yes)
+			)
+		)
+		(property "Description" "-55℃~+155℃ 0Ω 50V 62.5mW Thick Film Resistor ±1% ±800ppm/℃ 0402 Chip Resistor - Surface Mount ROHS"
+			(at 62.23 173.99 0)
+			(effects
+				(font
+					(size 1.27 1.27)
+				)
+				(hide yes)
+			)
+		)
+		(property "Resistance" "0"
+			(at 62.23 176.276 90)
+			(effects
+				(font
+					(size 1.27 1.27)
+				)
+			)
+		)
+		(property "LCSC" "C17168"
+			(at 62.23 173.99 0)
+			(effects
+				(font
+					(size 1.27 1.27)
+				)
+				(hide yes)
+			)
+		)
+		(pin "1"
+		)
+		(pin "2"
+		)
+		(instances
+			(project "NanoGaN"
+				(path "/aa8a494f-605e-4a00-9d3c-daec94709fcb/2aff88eb-0d92-4253-8876-ba05112be4d6"
+					(reference "R7")
+					(unit 1)
+				)

Commit message: couple of ERC fixes
Changed lines of the file:
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@@
 	)
 	(junction
+		(at 100.33 125.73)
+		(diameter 0)
+		(color 0 0 0 0)
+	)
+	(junction
 		(at 73.66 93.98)
 		(diameter 0)
@@
 	(wire
 		(pts
+			(xy 137.16 22.86) (xy 137.16 25.4)
+		)
+		(stroke
+			(width 0)
+			(type default)
+		)
+	)
+	(wire
+		(pts
 			(xy 38.1 137.16) (xy 38.1 139.7)
 		)
@@
 	(wire
 		(pts
+			(xy 100.33 123.19) (xy 100.33 125.73)
+		)
+		(stroke
+			(width 0)
+			(type default)
+		)
+	)
+	(wire
+		(pts
 			(xy 38.1 173.99) (xy 38.1 176.53)
 		)
@@
 	)
 	(symbol
+		(lib_id "power:PWR_FLAG")
+		(at 137.16 22.86 0)
+		(unit 1)
+		(exclude_from_sim no)
+		(in_bom yes)
+		(on_board yes)
+		(dnp no)
+		(property "Reference" "#FLG03"
+			(at 137.16 20.955 0)
+			(effects
+				(font
+					(size 1.27 1.27)
+				)
+				(hide yes)
+			)
+		)
+		(property "Value" "PWR_FLAG"
+			(at 137.414 19.05 0)
+			(effects
+				(font
+					(size 1.27 1.27)
+				)
+			)
+		)
+		(property "Footprint" ""
+			(at 137.16 22.86 0)
+			(effects
+				(font
+					(size 1.27 1.27)
+				)
+				(hide yes)
+			)
+		)
+		(property "Datasheet" "~"
+			(at 137.16 22.86 0)
+			(effects
+				(font
+					(size 1.27 1.27)
+				)
+				(hide yes)
+			)
+		)
+		(property "Description" ""
+			(at 137.16 22.86 0)
+			(effects
+				(font
+					(size 1.27 1.27)
+				)
+			)
+		)
+		(pin "1"
+		)
+		(instances
+			(project "NanoGaN"
+				(path "/aa8a494f-605e-4a00-9d3c-daec94709fcb/2aff88eb-0d92-4253-8876-ba05112be4d6"
+					(reference "#FLG03")
+					(unit 1)
+				)
+			)
+		)
+	)
+	(symbol
 		(lib_id "power:VDC")
 		(at 38.1 121.92 0)
@@
 					(unit 1)
 				)
+			)
+		)
+	)
+	(symbol
+		(lib_id "power:PWR_FLAG")
+		(at 100.33 123.19 0)
+		(unit 1)
+		(exclude_from_sim no)
+		(in_bom yes)
+		(on_board yes)
+		(dnp no)
+		(property "Reference" "#FLG01"
+			(at 100.33 121.285 0)
+			(effects
+				(font
+					(size 1.27 1.27)
+				)
+				(hide yes)
+			)
+		)
+		(property "Value" "PWR_FLAG"
+			(at 100.584 119.38 0)
+			(effects
+				(font
+					(size 1.27 1.27)
+				)
+			)
+		)
+		(property "Footprint" ""
+			(at 100.33 123.19 0)
+			(effects
+				(font
+					(size 1.27 1.27)
+				)
+				(hide yes)
+			)
+		)
+		(property "Datasheet" "~"
+			(at 100.33 123.19 0)
+			(effects
+				(font
+					(size 1.27 1.27)
+				)
+				(hide yes)
+			)
+		)
+		(property "Description" ""
+			(at 100.33 123.19 0)
+			(effects
+				(font
+					(size 1.27 1.27)
+				)
+			)
+		)
+		(pin "1"
+		)
+		(instances
+			(project "NanoGaN"
+				(path "/aa8a494f-605e-4a00-9d3c-daec94709fcb/2aff88eb-0d92-4253-8876-ba05112be4d6"
+					(reference "#FLG01")
+					(unit 1)
+				)
