File: power.kicad_sch (KiCad schematic)
At the start: 39 parts, among them U2 LMR51635XDDCR, U3 AMS1117

Commit message: schematic and PCB reviews are done, ready for release and first order.
Parts:
- removed C11, C12, C13, C14, C27, C35: EKYC800ELL471MK25S, NanoGaN:CP_Radial_D12.5mm_P5.00mm, symbol NanoGaN:C_Polarized_FZ1J221M1313
- added C11, C12, C13, C14, C27, C35: EKYC800ELL471MK25S, NanoGaN:CP_Radial_D12.5mm_P5.00mm, symbol Device:C_Polarized
- R60: value 0402WGF2200TCE -> 0402WGF5100TCE; LCSC C25091 -> C25123; Resistance 220 -> 510
- U2: LCSC C45262770 -> C42432812
Connections:
- net GND: now also C11.2, C12.2, C13.2, C14.2, C27.2, C35.2
- net U_DC: now also C11.1, C12.1, C13.1, C14.1, C27.1, C35.1
Other:
- company: (none) -> Eren Akbayin
- title: (none) -> NanoGaN

Commit message: gate driver change is complete
Parts:
- R4: value 0603WAF3902T5E -> NQ02WGF3902TCE; footprint Resistor_SMD:R_0603_1608Metric -> Resistor_SMD:R_0402_1005Metric; LCSC C23153 -> C965259
